Commit message: custom moveIt package for ur5e with laser scanner

File: include/urdf/line_scanner.xacro (robot description, xacro)
@@ -7,5 +7,5 @@
         <geometry>
           <!-- Define the geometry of the laser scanner (e.g., a cylinder) -->
-          <cylinder radius="0.05" length="0.2"/>
+          <cylinder radius="0.025" length="0.1"/>
         </geometry>
         <material name="laser_scanner_material"/>
@@ -14,5 +14,5 @@
         <geometry>
           <!-- Collision geometry -->
-          <cylinder radius="0.05" length="0.2"/>
+          <cylinder radius="0.025" length="0.2"/>
         </geometry>
       </collision>
@@ -22,6 +22,9 @@
       <parent link="${parent_link}"/>
       <child link="laser_scanner_link"/>
-      <origin xyz="${position}" rpy="0 0 0"/>
+      <origin xyz="${position}" rpy="0 -1.57 0"/>
     </joint>
+    <gazebo reference="laser_scanner_link">
+      <material>Gazebo/Red</material>
+    </gazebo>
           <!-- Define the laser sensor and attach the plugin -->
     <gazebo reference="laser_scanner_link">
@@ -33,6 +36,6 @@
               <samples>1000</samples>
               <resolution>1</resolution>
-              <min_angle>-1.57</min_angle>
-              <max_angle>1.57</max_angle>
+              <min_angle>-0.1</min_angle>
+              <max_angle>0.1</max_angle>
             </horizontal>
           </scan>
@@ -48,8 +51,40 @@
           <topicName>laser_scan</topicName>
           <frameName>laser_scanner_link</frameName>
-          <updateRate>30</updateRate> <!-- Rate in Hz -->
+          <updateRate>10</updateRate> <!-- Rate in Hz -->
         </plugin>
       </sensor>
     </gazebo>
   </xacro:macro>
+  <!-- Define the laser scanner macro -->
+  <xacro:macro name="welding_eff" params="parent_link position">
+    <link name="welding_eff_link">
+      <visual>
+        <geometry>
+          <!-- Define the geometry of the laser scanner (e.g., a cylinder) -->
+          <cylinder radius="0.005" length="0.15"/>
+        </geometry>
+        <material name="welding_eff_material"/>
+      </visual>
+      <collision>
+        <geometry>
+          <!-- Collision geometry -->
+          <cylinder radius="0.005" length="0.2"/>
+        </geometry>
+      </collision>
+    </link>
+    <gazebo reference="welding_eff_link">
+      <material>Gazebo/Blue</material>
+    </gazebo>
+    <joint name="cone_approx_joint" type="fixed">
+      <parent link="${parent_link}"/>
+      <child link="welding_eff_link"/>
+      <origin xyz="${position}" rpy="0 0 0"/>
+    </joint>
+    <link name="tcp_eff"/>
+    <joint name="tcp_eff_cone_joint" type="fixed">
+      <parent link="welding_eff_link"/>
+      <child link="tcp_eff"/>
+      <origin xyz="0 0 0" rpy="0 0 0"/>
+    </joint>
+  </xacro:macro>
 </robot>

File: include/urdf/ur5e_laser.xacro (robot description, xacro)
@@ -6,8 +6,8 @@
     <xacro:include filename="$(find alpaka_demo)/include/urdf/line_scanner.xacro"/>
     <!-- Declare necessary arguments -->
-    <xacro:arg name="joint_limit_params" default=""/>
-    <xacro:arg name="physical_params" default=""/>
-    <xacro:arg name="kinematics_params" default=""/>
-    <xacro:arg name="visual_params" default=""/>
+    <xacro:arg name="joint_limit_params" default="$(find ur_description)/config/ur5e/joint_limits.yaml"/>
+    <xacro:arg name="physical_params" default="$(find ur_description)/config/ur5e/physical_parameters.yaml"/>
+    <xacro:arg name="kinematics_params" default="$(find ur_description)/config/ur5e/default_kinematics.yaml"/>
+    <xacro:arg name="visual_params" default="$(find ur_description)/config/ur5e/visual_parameters.yaml"/>
     <xacro:arg name="transmission_hw_interface" default="hardware_interface/EffortJointInterface"/>
     <xacro:arg name="safety_limits" default="false"/>
@@ -33,4 +33,6 @@
     </joint>
     <!-- Use the laser scanner macro to attach it to a specific link -->
-    <xacro:laser_scanner parent_link="wrist_3_link" position="0 0.1 0.1"/>
+    <xacro:laser_scanner parent_link="tool0" position="0 -0.1 0"/>
+    <!-- Include the cone end-effector and attach to the flange -->
+    <xacro:welding_eff parent_link="tool0" position="0 0 0.01"/>
 </robot>
