Commit message: created ur10 w/ alpaka end-effector config and operational with simple pose detection.

File: alpaka_demo/include/urdf/laser_scanner.xacro (robot description, xacro)
@@ -48,5 +48,5 @@
         <range>
           <min>0.1</min>
-          <max>2</max>
+          <max>0.5</max>
           <resolution>0.01</resolution>
         </range>

File: alpaka_demo/include/urdf/line_scanner.xacro (robot description, xacro)
@@ -2,5 +2,5 @@
 <robot xmlns:xacro="http://wiki.ros.org/xacro">
   <!-- Define the laser scanner macro -->
-  <xacro:macro name="laser_scanner" params="parent_link position">
+  <xacro:macro name="laser_scanner" params="parent_link">
     <link name="laser_scanner_link">
     </link>
@@ -18,13 +18,13 @@
           <scan>
             <horizontal>
-              <samples>1000</samples>
+              <samples>100</samples>
               <resolution>1</resolution>
-              <min_angle>-0.474</min_angle>
-              <max_angle>0.474</max_angle>
+              <min_angle>-0.237</min_angle>
+              <max_angle>0.237</max_angle>
             </horizontal>
           </scan>
           <range>
-            <min>0.1</min>
-            <max>10.0</max>
+            <min>0.74</min>
+            <max>0.158</max>
             <resolution>0.01</resolution>
           </range>
@@ -48,5 +48,5 @@
   </xacro:macro>
   <!-- Define the laser scanner macro -->
-  <xacro:macro name="welding_eff" params="parent_link position">
+  <xacro:macro name="welding_eff" params="parent_link">
     <link name="welding_eff_link">
       <visual>
@@ -79,9 +79,27 @@
       <origin rpy="0 1.57 0" xyz="0.05 0 0" />
     </joint>
-    <link name="tcp_eff"/>
+    <link name="tcp_eff">
+      <visual>
+        <origin xyz="0 0 0" rpy="0 0 0" />
+        <geometry>
+          <sphere radius="0.005"/>
+        </geometry>
+      </visual>
+      <collision>
+        <origin xyz="0 0 0" rpy="0 0 0" />
+        <geometry>
+          <sphere radius="0.005"/>
+        </geometry>
+      </collision>
+     <inertial>
+        <mass value="1e-6" />
+        <origin xyz="0 0 0" rpy="0 0 0" />
+        <inertia ixx="1e-6" iyy="1e-6" izz="1e-6" ixy="0.0" ixz="0.0" iyz="0.0" />
+      </inertial>
+    </link>
     <joint name="tcp_eff_joint" type="fixed">
       <parent link="welding_eff_link"/>
       <child link="tcp_eff"/>
-      <origin rpy="0 0.68 0" xyz="0.04561 0 0.61858" />
+      <origin rpy="1.5707 -0.8907 0" xyz="0.04561 0 0.61858" />
     </joint>
   </xacro:macro>

File: alpaka_demo/include/urdf/ur10e_alpaka.xacro (robot description, xacro)
@@ -1,4 +1,4 @@
 <?xml version="1.0"?>
-<robot xmlns:xacro="http://wiki.ros.org/xacro" name="ur5e_laser_robot">
+<robot xmlns:xacro="http://wiki.ros.org/xacro" name="ur10e_alpaka">
     <!-- Include the UR5e Gazebo-compatible Xacro -->
     <xacro:include filename="$(find ur_gazebo)/urdf/ur_macro.xacro"/>
@@ -6,8 +6,8 @@
     <xacro:include filename="$(find alpaka_demo)/include/urdf/line_scanner.xacro"/>
     <!-- Declare necessary arguments -->
-    <xacro:arg name="joint_limit_params" default="$(find ur_description)/config/ur5e/joint_limits.yaml"/>
-    <xacro:arg name="physical_params" default="$(find ur_description)/config/ur5e/physical_parameters.yaml"/>
-    <xacro:arg name="kinematics_params" default="$(find ur_description)/config/ur5e/default_kinematics.yaml"/>
-    <xacro:arg name="visual_params" default="$(find ur_description)/config/ur5e/visual_parameters.yaml"/>
+    <xacro:arg name="joint_limit_params" default="$(find ur_description)/config/ur10e/joint_limits.yaml"/>
+    <xacro:arg name="physical_params" default="$(find ur_description)/config/ur10e/physical_parameters.yaml"/>
+    <xacro:arg name="kinematics_params" default="$(find ur_description)/config/ur10e/default_kinematics.yaml"/>
+    <xacro:arg name="visual_params" default="$(find ur_description)/config/ur10e/visual_parameters.yaml"/>
     <xacro:arg name="transmission_hw_interface" default="hardware_interface/EffortJointInterface"/>
     <xacro:arg name="safety_limits" default="false"/>

File: ur10e_alpaka/config/gazebo_ur10e_alpaka.urdf (robot description, URDF)
Before this commit: robot ur5e_laser_robot, 14 links, 13 joints
Links:
- added link tool0
- link base_link_inertia: geometry collision mesh filename=package://ur_description/meshes/ur10e/collision/base.stl; visual mesh filename=package://ur_description/meshes/ur10e/visual/base.dae
- link forearm_link: mass 2.275 -> 3.87; geometry collision mesh filename=package://ur_description/meshes/ur10e/collision/forearm.stl; visual mesh filename=package://ur_description/meshes/ur10e/visual/forearm.dae
- link shoulder_link: mass 3.7 -> 7.778; geometry collision mesh filename=package://ur_description/meshes/ur10e/collision/shoulder.stl; visual mesh filename=package://ur_description/meshes/ur10e/visual/shoulder.dae
- link upper_arm_link: mass 8.393 -> 12.93; geometry collision mesh filename=package://ur_description/meshes/ur10e/collision/upperarm.stl; visual mesh filename=package://ur_description/meshes/ur10e/visual/upperarm.dae
- link wrist_1_link: mass 1.219 -> 1.96; geometry collision mesh filename=package://ur_description/meshes/ur10e/collision/wrist1.stl; visual mesh filename=package://ur_description/meshes/ur10e/visual/wrist1.dae
- link wrist_2_link: mass 1.219 -> 1.96; geometry collision mesh filename=package://ur_description/meshes/ur10e/collision/wrist2.stl; visual mesh filename=package://ur_description/meshes/ur10e/visual/wrist2.dae
- link wrist_3_link: mass 0.1879 -> 0.202; geometry collision mesh filename=package://ur_description/meshes/ur10e/collision/wrist3.stl; visual mesh filename=package://ur_description/meshes/ur10e/visual/wrist3.dae
Joints:
- added joint flange-tool0: type fixed, parent flange, child tool0, origin xyz=0 0 0 rpy=1.5707963267948966 0 1.5707963267948966
- joint elbow_joint: origin xyz=-0.425 0 0 rpy=0 0 0 -> xyz=-0.6127 0 0 rpy=0 0 0
- joint shoulder_lift_joint: limit lower=-6.283185307179586 upper=6.283185307179586 effort=150.0 velocity=3.141592653589793 -> lower=-6.283185307179586 upper=6.283185307179586 effort=330.0 velocity=2.0943951023931953
- joint shoulder_pan_joint: limit lower=-6.283185307179586 upper=6.283185307179586 effort=150.0 velocity=3.141592653589793 -> lower=-6.283185307179586 upper=6.283185307179586 effort=330.0 velocity=2.0943951023931953; origin xyz=0 0 0.1625 rpy=0 0 0 -> xyz=0 0 0.1807 rpy=0 0 0
- joint tcp_eff_joint: origin xyz=0.04561 0 0.61858 rpy=0 0.68 0 -> xyz=0.04561 0 0.61858 rpy=1.5707 -0.8907 0
- joint wrist_1_joint: limit lower=-6.283185307179586 upper=6.283185307179586 effort=28.0 velocity=3.141592653589793 -> lower=-6.283185307179586 upper=6.283185307179586 effort=56.0 velocity=3.141592653589793; origin xyz=-0.3922 0 0.1333 rpy=0 0 0 -> xyz=-0.57155 0 0.17415 rpy=0 0 0
- joint wrist_2_joint: limit lower=-6.283185307179586 upper=6.283185307179586 effort=28.0 velocity=3.141592653589793 -> lower=-6.283185307179586 upper=6.283185307179586 effort=56.0 velocity=3.141592653589793; origin xyz=0 -0.0997 -2.044881182297852e-11 rpy=1.570796327 0 0 -> xyz=0 -0.11985 -2.458164590756244e-11 rpy=1.570796327 0 0
- joint wrist_3_joint: limit lower=-6.283185307179586 upper=6.283185307179586 effort=28.0 velocity=3.141592653589793 -> lower=-6.283185307179586 upper=6.283185307179586 effort=56.0 velocity=3.141592653589793; origin xyz=0 0.0996 -2.042830148012698e-11 rpy=1.570796326589793 3.141592653589793 3.141592653589793 -> xyz=0 0.11655 -2.390480459346185e-11 rpy=1.570796326589793 3.141592653589793 3.141592653589793
