Commit message: testing pose orientation

File: alpaka_demo/include/urdf/line_scanner.xacro (robot description, xacro)
@@ -5,7 +5,8 @@
     <link name="laser_scanner_link">
       <visual>
+      <origin xyz="0 0 0" rpy="1.57 0 0" />
         <geometry>
           <!-- Define the geometry of the laser scanner (e.g., a cylinder) -->
-          <cylinder radius="0.025" length="0.1"/>
+          <cylinder radius="0.015" length="0.1"/>
         </geometry>
         <material name="laser_scanner_material"/>
@@ -14,7 +15,12 @@
         <geometry>
           <!-- Collision geometry -->
-          <cylinder radius="0.025" length="0.2"/>
+          <cylinder radius="0.015" length="0.2"/>
         </geometry>
       </collision>
+      <inertial>
+            <mass value="1e-6" />
+            <origin xyz="0 0 0" rpy="1.57 0 0" />
+            <inertia ixx="1e-6" iyy="1e-6" izz="1e-6" ixy="0.0" ixz="0.0" iyz="0.0" />
+      </inertial>
     </link>
     <!-- Attach the laser scanner to a parent link -->
@@ -22,5 +28,5 @@
       <parent link="${parent_link}"/>
       <child link="laser_scanner_link"/>
-      <origin xyz="${position}" rpy="0 -1.57 0"/>
+      <origin xyz="${position}" rpy="0 0 0"/>
     </joint>
     <gazebo reference="laser_scanner_link">
@@ -36,6 +42,6 @@
               <samples>1000</samples>
               <resolution>1</resolution>
-              <min_angle>-0.1</min_angle>
-              <max_angle>0.1</max_angle>
+              <min_angle>-0.474</min_angle>
+              <max_angle>0.474</max_angle>
             </horizontal>
           </scan>
@@ -72,4 +78,9 @@
         </geometry>
       </collision>
+      <inertial>
+            <mass value="1e-6" />
+            <origin xyz="0 0 0" rpy="0 0 0" />
+            <inertia ixx="1e-6" iyy="1e-6" izz="1e-6" ixy="0.0" ixz="0.0" iyz="0.0" />
+      </inertial>
     </link>
     <gazebo reference="welding_eff_link">
@@ -79,5 +90,5 @@
       <parent link="${parent_link}"/>
       <child link="welding_eff_link"/>
-      <origin xyz="${position}" rpy="0 0 0"/>
+      <origin xyz="${position}" rpy="0 1.57 0"/>
     </joint>
     <link name="tcp_eff"/>

File: alpaka_demo/include/urdf/ur5e_laser.xacro (robot description, xacro)
@@ -33,6 +33,6 @@
     </joint>
     <!-- Use the laser scanner macro to attach it to a specific link -->
-    <xacro:laser_scanner parent_link="flange" position="0 -0.1 0"/>
+    <xacro:laser_scanner parent_link="flange" position="0 0 -0.05"/>
     <!-- Include the cone end-effector and attach to the flange -->
-    <xacro:welding_eff parent_link="flange" position="0 0 0.01"/>
+    <xacro:welding_eff parent_link="flange" position="0 0 0"/>
 </robot>

Commit message: tcp corrected

File: alpaka_demo/include/urdf/line_scanner.xacro (robot description, xacro)
@@ -15,5 +15,5 @@
         <geometry>
           <!-- Collision geometry -->
-          <cylinder radius="0.015" length="0.2"/>
+          <cylinder radius="0.015" length="0.1"/>
         </geometry>
       </collision>
@@ -66,14 +66,16 @@
     <link name="welding_eff_link">
       <visual>
+      <origin xyz="-0.025 0 0.0" rpy="0 0 0" />
         <geometry>
           <!-- Define the geometry of the laser scanner (e.g., a cylinder) -->
-          <cylinder radius="0.005" length="0.15"/>
+          <cylinder radius="0.005" length="0.05"/>
         </geometry>
         <material name="welding_eff_material"/>
       </visual>
       <collision>
+        <origin xyz="-0.025 0 0.0" rpy="0 0 0" />
         <geometry>
           <!-- Collision geometry -->
-          <cylinder radius="0.005" length="0.2"/>
+          <cylinder radius="0.005" length="0.05"/>
         </geometry>
       </collision>

File: ur5e_laser_sim/config/gazebo_ur5e_laser_robot.urdf (robot description, URDF)
Before this commit: robot ur5e_laser_robot, 14 links, 13 joints
Links:
- link welding_eff_link: geometry collision cylinder length=0.05 radius=0.005; visual cylinder length=0.05 radius=0.005
Joints:
- joint cone_approx_joint: origin xyz=0 0 0 rpy=0 1.57 0 -> xyz=0.05 0 0.0 rpy=0 1.57 0

Commit message: added welding eff and line scanner to model

File: alpaka_demo/include/urdf/line_scanner.xacro (robot description, xacro)
@@ -66,17 +66,13 @@
     <link name="welding_eff_link">
       <visual>
-      <origin xyz="-0.025 0 0.0" rpy="0 0 0" />
+      <origin xyz="0 0 0" rpy="0 0 0" />
         <geometry>
-          <!-- Define the geometry of the laser scanner (e.g., a cylinder) -->
-          <cylinder radius="0.005" length="0.05"/>
-        </geometry>
-        <material name="welding_eff_material"/>
-      </visual>
-      <collision>
-        <origin xyz="-0.025 0 0.0" rpy="0 0 0" />
-        <geometry>
-          <!-- Collision geometry -->
-          <cylinder radius="0.005" length="0.05"/>
-        </geometry>
+                <mesh filename="package://alpaka_demo/include/urdf/meshes/welding_eff/Brennerhalter_with_Sensor.dae"/>
+            </geometry>
+        </visual>
+        <collision>
+            <geometry>
+                <mesh filename="package://alpaka_demo/include/urdf/meshes/welding_eff/Brennerhalter_with_Sensor.stl"/>
+            </geometry>
       </collision>
       <inertial>
@@ -92,5 +88,5 @@
       <parent link="${parent_link}"/>
       <child link="welding_eff_link"/>
-      <origin xyz="${position}" rpy="0 1.57 0"/>
+      <origin xyz="${position}" rpy="3.14 -1.57 0"/>
     </joint>
     <link name="tcp_eff"/>

File: ur5e_laser_sim/config/gazebo_ur5e_laser_robot.urdf (robot description, URDF)
Before this commit: robot ur5e_laser_robot, 14 links, 13 joints
Links:
- link welding_eff_link: geometry collision mesh filename=package://alpaka_demo/include/urdf/meshes/welding_eff/Brenn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; visual mesh filename=package://alpaka_demo/include/urdf/meshes/welding_eff/Brenn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
Joints:
- joint cone_approx_joint: origin xyz=0.05 0 0.0 rpy=0 1.57 0 -> xyz=0.05 0 0.0 rpy=3.14 -1.57 0

Commit message: end-effector orientated but laser scanning not working

File: alpaka_demo/include/urdf/line_scanner.xacro (robot description, xacro)
@@ -82,11 +82,8 @@
       </inertial>
     </link>
-    <gazebo reference="welding_eff_link">
-      <material>Gazebo/Blue</material>
-    </gazebo>
-    <joint name="cone_approx_joint" type="fixed">
+    <joint name="welding_eff_joint" type="fixed">
       <parent link="${parent_link}"/>
       <child link="welding_eff_link"/>
-      <origin xyz="${position}" rpy="3.14 -1.57 0"/>
+      <origin xyz="${position}" rpy="0 1.57 0"/>
     </joint>
     <link name="tcp_eff"/>

File: ur5e_laser_sim/config/gazebo_ur5e_laser_robot.urdf (robot description, URDF)
Before this commit: robot ur5e_laser_robot, 14 links, 13 joints
Links:
- link laser_scanner_link: mass 1e-6 -> None; geometry 
Joints:
- removed joint cone_approx_joint
- added joint welding_eff_joint: type fixed, parent flange, child welding_eff_link, origin xyz=0.05 0 0 rpy=0 1.57 0
- joint laser_scanner_joint: origin xyz=0 0 -0.05 rpy=0 0 0 -> xyz=-0.02684 0.07237 0.52914 rpy=0 0 0; parent flange -> welding_eff_link

Commit message: deactivated collision mesh

File: alpaka_demo/include/urdf/line_scanner.xacro (robot description, xacro)
@@ -4,23 +4,4 @@
   <xacro:macro name="laser_scanner" params="parent_link position">
     <link name="laser_scanner_link">
-      <visual>
-      <origin xyz="0 0 0" rpy="1.57 0 0" />
-        <geometry>
-          <!-- Define the geometry of the laser scanner (e.g., a cylinder) -->
-          <cylinder radius="0.015" length="0.1"/>
-        </geometry>
-        <material name="laser_scanner_material"/>
-      </visual>
-      <collision>
-        <geometry>
-          <!-- Collision geometry -->
-          <cylinder radius="0.015" length="0.1"/>
-        </geometry>
-      </collision>
-      <inertial>
-            <mass value="1e-6" />
-            <origin xyz="0 0 0" rpy="1.57 0 0" />
-            <inertia ixx="1e-6" iyy="1e-6" izz="1e-6" ixy="0.0" ixz="0.0" iyz="0.0" />
-      </inertial>
     </link>
     <!-- Attach the laser scanner to a parent link -->
@@ -28,9 +9,6 @@
       <parent link="${parent_link}"/>
       <child link="laser_scanner_link"/>
-      <origin xyz="${position}" rpy="0 0 0"/>
+      <origin rpy="0 -0.890118 -0.28797" xyz="-0.02684 0.07237 0.52914"/>
     </joint>
-    <gazebo reference="laser_scanner_link">
-      <material>Gazebo/Red</material>
-    </gazebo>
           <!-- Define the laser sensor and attach the plugin -->
     <gazebo reference="laser_scanner_link">
@@ -51,4 +29,11 @@
             <resolution>0.01</resolution>
           </range>
+          <collision>
+            <surface>
+              <contact>
+                <collide_bitmask>0b01</collide_bitmask> <!-- Set bitmask -->
+              </contact>
+            </surface>
+          </collision>
         </ray>
         <!-- Add Gazebo Laser Scanner Plugin -->
@@ -66,13 +51,20 @@
     <link name="welding_eff_link">
       <visual>
-      <origin xyz="0 0 0" rpy="0 0 0" />
+        <origin xyz="0 0 -0.05" rpy="0 0 0" />
         <geometry>
                 <mesh filename="package://alpaka_demo/include/urdf/meshes/welding_eff/Brennerhalter_with_Sensor.dae"/>
             </geometry>
         </visual>
-        <collision>
-            <geometry>
-                <mesh filename="package://alpaka_demo/include/urdf/meshes/welding_eff/Brennerhalter_with_Sensor.stl"/>
-            </geometry>
+      <collision>
+        <origin xyz="0 0 -0.05" rpy="0 0 0" />
+        <geometry>
+          <mesh filename="package://alpaka_demo/include/urdf/meshes/welding_eff/Brennerhalter_with_Sensor.stl"/>
+        </geometry>
+        <laser_retro>0</laser_retro> <!-- Makes the collision invisible to laser rays -->
+        <surface>
+          <contact>
+            <collide_bitmask>0b10</collide_bitmask> <!-- Set bitmask -->
+          </contact>
+        </surface>
       </collision>
       <inertial>
@@ -85,11 +77,11 @@
       <parent link="${parent_link}"/>
       <child link="welding_eff_link"/>
-      <origin xyz="${position}" rpy="0 1.57 0"/>
+      <origin rpy="0 1.57 0" xyz="0.05 0 0" />
     </joint>
     <link name="tcp_eff"/>
-    <joint name="tcp_eff_cone_joint" type="fixed">
+    <joint name="tcp_eff_joint" type="fixed">
       <parent link="welding_eff_link"/>
       <child link="tcp_eff"/>
-      <origin xyz="0 0 0" rpy="0 0 0"/>
+      <origin rpy="0 0.68 0" xyz="0.04561 0 0.61858" />
     </joint>
   </xacro:macro>

File: ur5e_laser_sim/config/gazebo_ur5e_laser_robot.urdf (robot description, URDF)
Before this commit: robot ur5e_laser_robot, 14 links, 13 joints
Links:
- link welding_eff_link: geometry visual mesh filename=package://alpaka_demo/include/urdf/meshes/welding_eff/Brenn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
Joints:
- joint laser_scanner_joint: origin xyz=-0.02684 0.07237 0.52914 rpy=0 -0.890118 -0.28797 -> xyz=-0.02684 0.07237 0.52914 rpy=1.57 -0.890118 -0.28797

Commit message: laser matches alpaka sensor positioning

File: alpaka_demo/include/urdf/line_scanner.xacro (robot description, xacro)
@@ -9,10 +9,10 @@
       <parent link="${parent_link}"/>
       <child link="laser_scanner_link"/>
-      <origin rpy="0 -0.890118 -0.28797" xyz="-0.02684 0.07237 0.52914"/>
+      <origin rpy="1.8587757 -0.890118 -0.2879793" xyz="-0.02684 0.07237 0.52914" />
     </joint>
           <!-- Define the laser sensor and attach the plugin -->
     <gazebo reference="laser_scanner_link">
       <sensor type="ray" name="laser_scan">
-        <origin xyz="${position}" />
+        <origin xyz="0 0 0" rpy="0 0 0"/>
         <ray>
           <scan>

File: alpaka_demo/include/urdf/ur5e_laser.xacro (robot description, xacro)
@@ -32,7 +32,7 @@
         <origin xyz="0 0 0" rpy="0 0 0"/>
     </joint>
-    <!-- Use the laser scanner macro to attach it to a specific link -->
-    <xacro:laser_scanner parent_link="flange" position="0 0 -0.05"/>
     <!-- Include the cone end-effector and attach to the flange -->
     <xacro:welding_eff parent_link="flange" position="0 0 0"/>
+    <!-- Use the laser scanner macro to attach it to a specific link -->
+    <xacro:laser_scanner parent_link="welding_eff_link" position="0 0 -0.05"/>
 </robot>

File: ur5e_laser_sim/config/gazebo_ur5e_laser_robot.urdf (robot description, URDF)
Before this commit: robot ur5e_laser_robot, 14 links, 13 joints
Joints:
- joint laser_scanner_joint: origin xyz=-0.02684 0.07237 0.52914 rpy=1.57 -0.890118 -0.28797 -> xyz=-0.02684 0.07237 0.52914 rpy=1.8587757 -0.890118 -0.2879793

Commit message: updated laser scanner orientation for scan across x/z plane

File: alpaka_demo/include/urdf/line_scanner.xacro (robot description, xacro)
@@ -28,5 +28,5 @@
       <parent link="${parent_link}"/>
       <child link="laser_scanner_link"/>
-      <origin xyz="${position}" rpy="0 0 0"/>
+      <origin xyz="${position}" rpy="1.5708 0 1.5708"/>
     </joint>
     <gazebo reference="laser_scanner_link">
@@ -36,5 +36,5 @@
     <gazebo reference="laser_scanner_link">
       <sensor type="ray" name="laser_scan">
-        <origin xyz="${position}" />
+        <pose>0 0 0 -1.5708 -1.5708 0</pose>
         <ray>
           <scan>
@@ -42,6 +42,6 @@
               <samples>1000</samples>
               <resolution>1</resolution>
-              <min_angle>-0.474</min_angle>
-              <max_angle>0.474</max_angle>
+              <min_angle>-0.1937</min_angle>
+              <max_angle>0.1937</max_angle>
             </horizontal>
           </scan>

File: ur5e_laser_sim/config/gazebo_ur5e_laser_robot.urdf (robot description, URDF)
Before this commit: robot ur5e_laser_robot, 14 links, 13 joints
Joints:
- joint laser_scanner_joint: origin xyz=-0.025 0 -0.05 rpy=0 0 0 -> xyz=-0.025 0 -0.05 rpy=1.5708 0 1.5708

File: ur5e_laser_sim/config/noise_ur5e_laser_robot.urdf (robot description, URDF)
Before this commit: robot ur5e_laser_robot, 14 links, 13 joints
Joints:
- joint laser_scanner_joint: origin xyz=-0.025 0 -0.05 rpy=0 0 0 -> xyz=-0.025 0 -0.05 rpy=1.5708 0 1.5708

Commit message: update laser cylinder rotation

File: alpaka_demo/include/urdf/line_scanner.xacro (robot description, xacro)
@@ -5,5 +5,5 @@
     <link name="laser_scanner_link">
       <visual>
-      <origin xyz="0 0 0" rpy="1.57 0 0" />
+      <origin xyz="0 0 0" rpy="0 0 0" />
         <geometry>
           <!-- Define the geometry of the laser scanner (e.g., a cylinder) -->
