Commit message: custom moveit ur5e with laser scanner operational. Laser in wrong orientation.

File: ur5e_laser_sim/config/gazebo_ur5e_laser_robot.urdf (robot description, URDF)
Before this commit: robot ur5e_laser_robot, 15 links, 14 joints
Links:
- removed link tool0
- link laser_scanner_link: geometry collision cylinder length=0.2 radius=0.015; visual cylinder length=0.1 radius=0.015
Joints:
- removed joint flange-tool0
- joint cone_approx_joint: origin xyz=0 0 0.01 rpy=0 0 0 -> xyz=0 0 0 rpy=0 1.57 0; parent tool0 -> flange
- joint laser_scanner_joint: origin xyz=0 -0.1 0 rpy=0 -1.57 0 -> xyz=0 0 -0.05 rpy=1.57 0 0; parent tool0 -> flange

Commit message: scanner orientation corrected

File: ur5e_laser_sim/config/gazebo_ur5e_laser_robot.urdf (robot description, URDF)
Before this commit: robot ur5e_laser_robot, 14 links, 13 joints
Joints:
- joint laser_scanner_joint: origin xyz=0 0 -0.05 rpy=1.57 0 0 -> xyz=0 0 -0.05 rpy=0 0 0

Commit message: robot movement towards pose but wrist_3 error is present

File: ur5e_laser_sim/config/gazebo_ur5e_laser_robot.urdf (robot description, URDF)
Before this commit: robot ur5e_laser_robot, 14 links, 13 joints
Links:
- link laser_scanner_link: mass 0.1 -> 1e-6
- link welding_eff_link: mass 0.1 -> 1e-6

Commit message: robot moves to a detected seam

File: ur5e_laser_sim/config/gazebo_ur5e_laser_robot.urdf (robot description, URDF)
Before this commit: robot ur5e_laser_robot, 14 links, 13 joints
Links:
- link laser_scanner_link: geometry collision cylinder length=0.1 radius=0.015; visual cylinder length=0.1 radius=0.015
- link welding_eff_link: geometry collision cylinder length=0.15 radius=0.005; visual cylinder length=0.15 radius=0.005

Commit message: moved laser sensor position

File: ur5e_laser_sim/config/gazebo_ur5e_laser_robot.urdf (robot description, URDF)
Before this commit: robot ur5e_laser_robot, 14 links, 13 joints
Joints:
- joint laser_scanner_joint: origin xyz=0 0 -0.05 rpy=0 0 0 -> xyz=-0.025 0 -0.05 rpy=0 0 0

Commit message: alpaka scanner corrected orientation

File: ur5e_laser_sim/config/gazebo_ur5e_laser_robot.urdf (robot description, URDF)
Before this commit: robot ur5e_laser_robot, 14 links, 13 joints
Joints:
- removed joint tcp_eff_cone_joint
- added joint tcp_eff_joint: type fixed, parent welding_eff_link, child tcp_eff, origin xyz=0.04561 0 0.61858 rpy=0 0.68 0
- joint laser_scanner_joint: origin xyz=-0.02684 0.07237 0.52914 rpy=0 0 0 -> xyz=-0.02684 0.07237 0.52914 rpy=0 -0.890118 -0.28797

Commit message: robot control operation and camera tilted.

File: ur5e_laser_sim/config/gazebo_ur5e_laser_robot.urdf (robot description, URDF)
Before this commit: robot ur5e_laser_robot, 14 links, 13 joints
Joints:
- joint laser_scanner_joint: origin xyz=-0.025 0 -0.05 rpy=0 0 0 -> xyz=-0.025 0 -0.05 rpy=0 -0.2879793 0

Commit message: update config and launch file files

File: ur5e_laser_sim/config/gazebo_ur5e_laser_robot.urdf (robot description, URDF)
Before this commit: robot ur5e_laser_robot, 14 links, 13 joints
Joints:
- joint laser_scanner_joint: origin xyz=-0.025 0 -0.05 rpy=0 -0.2879793 0 -> xyz=-0.025 0 -0.05 rpy=0 0 0

Commit message: update laser orientation

File: ur5e_laser_sim/config/gazebo_ur5e_laser_robot.urdf (robot description, URDF)
Before this commit: robot ur5e_laser_robot, 14 links, 13 joints
Joints:
- joint laser_scanner_joint: origin xyz=-0.025 0 -0.05 rpy=0 0 0 -> xyz=-0.025 0 -0.05 rpy=1.5708 0 1.5708
